File: inputs_temp.sch (KiCad schematic (older format))
At the start: 10 parts

Commit message: Primer version
Esquematico completo, faltan notas del revisor.
Parts:
- removed C?: 1uF, symbol C
- removed L?: BLM18PG471SN1D, symbol L_Core_Ferrite
- removed U?: MAX31855KASA+, symbol MAX31855KASA+
- added C2, C8: 100n, footprints:C_0603_HandSoldering, symbol C
- added C5, C7: 10u, footprints:C_0603_HandSoldering, symbol C
- added J1, J2, J3: Screw_Terminal_1x02, footprints:TerminalBlock_Pheonix_MKDS1.5-2pol, symbol Screw_Terminal_1x02
- added L2: BLM18PG471SN1D, footprints:C_0603_HandSoldering, symbol L_Core_Ferrite
- added U1: NUP2105LT1G, footprints:SC-59_Handsoldering, symbol NUP2105LT1G
- added U2: MAX31855KASA+, footprints:SOIC-8, symbol MAX31855KASA+
- added U4: SN74LVC2G34DBVR, footprints:SOT-23-6_Handsoldering, symbol SN74LVC2G34DBVR
- C1: renamed from C?; value C -> NM; footprint (none) -> footprints:C_0603_HandSoldering; Description (none) -> Value; Digikey# (none) -> Value; Manf (none) -> Value; Manf# (none) -> Value; Mouser# (none) -> Value
- C3: renamed from C?; value C -> NM; footprint (none) -> footprints:C_0603_HandSoldering; Digikey# (none) -> Value; Manf (none) -> Value; Manf# (none) -> Value; Mouser# (none) -> Value
- C4: renamed from C?; footprint (none) -> footprints:C_0603_HandSoldering; Description (none) -> 10µF -20%, +80% 10V Ceramic Capacitor Y5V; Digikey# Value -> 311-1355-2-ND; Manf Value -> Yageo; Manf# Value -> CC0805ZKY5V6BB106; Mouser# Value -> 603-CC805ZKY5V6BB106
- C6: renamed from C?; footprint (none) -> footprints:C_0603_HandSoldering; Description (none) -> Value; Manf Value -> Yageo; Manf# Value -> CC0603KRX7R7BB104; Mouser# Value -> 603-CC603KRX7R7BB104
- L1: renamed from L?; footprint (none) -> footprints:C_0603_HandSoldering; Description (none) -> Ferrite Beads 470 OHM; Manf Value -> Murata Electronics; Manf# Value -> BLM18PG471SN1D; Mouser# Value -> 81-BLM18PG471SN1D
- R1: renamed from R?; value 100k -> 10k; footprint (none) -> footprints:R_1206_HandSoldering; Description (none) -> 10k Ohm ±5% 0.25W, 1/4W Chip, Moisture Resistant Thick Film; Digikey# Value -> 311-10KERTR-ND; Manf Value -> Yageo; Manf# Value -> RC1206JR-0710KL
- U3: renamed from U?; Description (none) -> Operational Amplifiers - Op Amps Single 2.7V; Digikey# (none) -> Value; Manf (none) -> Microchip Technology; Manf# (none) -> MCP601T-I/OT; Mouser# (none) -> 579-MCP601T-I/OT
Connections:
- net labels added: +3.3V, ADC_TERM, MISO_TCUP, SCK_TCUP, SS_TCUP
- net labels removed: +3,3V
- wire segments 17 -> 69
- no-connect marks 0 -> 1
Other:
- note added: "Entrada Termocupla"
- note added: "Entrada Termoresistor"
- note added: "Resistor de Referencia"
- moved on the sheet: C1, C3, C4, C6, L1, R1, U3
