File: inputs_temp.sch (KiCad schematic (older format))
At the start: 13 parts, among them J1 Screw_Terminal_1x02, J2 Screw_Terminal_1x02, J3 Screw_Terminal_1x02, U1 NUP2105LT1G, U2 MAX31855KASA+, U3 MCP601R

Commit message: Primer version del PCB
Se agregan modificaciones segun primer correccion. Se carga primer version  del PCB.
Parts:
- removed C7: 10u, footprints:C_0603_HandSoldering, symbol C
- removed C8: 100n, footprints:C_0603_HandSoldering, symbol C
- added C1, C3: 10u, footprints:C_0805_HandSoldering, symbol C
- C2, C6: footprint footprints:C_0603_HandSoldering -> footprints:C_0805_HandSoldering; Description Value -> Multilayer Ceramic Capacitors MLCC - SMD/SMT 0.1uF 10Volts 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; Digikey# Value -> 490-11592-1-ND; Manf Yageo -> Murata; Manf# CC0603KRX7R7BB104 -> GRM21B7U1A104JA01L; Mouser# 603-CC603KRX7R7BB104 -> 81-GRM21B7U1A104JA1L
- C4: footprint footprints:C_0603_HandSoldering -> footprints:C_0805_HandSoldering; Description 10µF -20%, +80% 10V Ceramic Capacitor Y5V -> Multilayer Ceramic Capacitors MLCC - SMD/SMT 0805 10uF 6.3v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; Digikey# 311-1355-2-ND -> 490-1718-1-ND; Manf Yageo -> Murata; Manf# CC0805ZKY5V6BB106 -> GRM21BR60J106ME19L; Mouser# 603-CC805ZKY5V6BB106 -> 81-GRM21BR60J106ME19
- C5: value 10u -> 100n; footprint footprints:C_0603_HandSoldering -> footprints:C_0805_HandSoldering; Description 10µF -20%, +80% 10V Ceramic Capacitor Y5V -> Multilayer Ceramic Capacitors MLCC - SMD/SMT 0.1uF 10Volts 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; Digikey# 311-1355-2-ND -> 490-11592-1-ND; Manf Yageo -> Murata; Manf# CC0805ZKY5V6BB106 -> GRM21B7U1A104JA01L; Mouser# 603-CC805ZKY5V6BB106 -> 81-GRM21B7U1A104JA1L
- R1: footprint footprints:R_1206_HandSoldering -> footprints:R_0805_HandSoldering; Description 10k Ohm ±5% 0.25W, 1/4W Chip, Moisture Resistant Thick Film -> Thick Film Resistors - SMD 10K OHM 1%; Digikey# 311-10KERTR-ND -> 311-10.0KCRCT-ND; Manf# RC1206JR-0710KL -> RC0805FR-0710KL; Mouser# Value -> 603-RC0805FR-0710KL
Connections:
- net GND: now also C1.1, C3.1
- net at R1.1, U3.3 (+): now also C1.2; no longer C5.2
- net +3.3V renamed +3V3
- net +3V3: now also C5.2, C3.2
- net GNDA_TERM renamed GNDA

Commit message: Correccion Final
Se trabajo sobre correcciones de 2da revision. Se agregaron archivos gerbers, BOM, y objetos 3D
Parts:
- U1: footprint footprints:SC-59_Handsoldering -> footprints:SOT23_NPN
Changed lines of the file:
@@
 EESchema Schematic File Version 2
 LIBS:TempRelay
-LIBS:power
-LIBS:tempRelayPoncho-cache
 EELAYER 25 0
 EELAYER END
@@
 $EndComp
 $Comp
-L GND #PWR016
+L GND #PWR015
 U 1 1 594B0304
 P 5100 1600
-F 0 "#PWR016" H 5100 1350 50  0001 C CNN
+F 0 "#PWR015" H 5100 1350 50  0001 C CNN
 F 1 "GND" H 5100 1450 50  0000 C CNN
 F 2 "" H 5100 1600 50  0001 C CNN
@@
 $EndComp
 $Comp
-L GND #PWR017
+L GND #PWR016
 U 1 1 594B0325
 P 6000 2550
-F 0 "#PWR017" H 6000 2300 50  0001 C CNN
+F 0 "#PWR016" H 6000 2300 50  0001 C CNN
 F 1 "GND" H 6000 2400 50  0000 C CNN
 F 2 "" H 6000 2550 50  0001 C CNN
@@
 $EndComp
 $Comp
-L GND #PWR018
+L GND #PWR017
 U 1 1 594B033F
 P 5100 2800
-F 0 "#PWR018" H 5100 2550 50  0001 C CNN
+F 0 "#PWR017" H 5100 2550 50  0001 C CNN
 F 1 "GND" H 5100 2650 50  0000 C CNN
 F 2 "" H 5100 2800 50  0001 C CNN
@@
 	6000 2550 6000 2500
 $Comp
-L GND #PWR019
+L GND #PWR018
 U 1 1 594B1832
 P 5700 5400
-F 0 "#PWR019" H 5700 5150 50  0001 C CNN
+F 0 "#PWR018" H 5700 5150 50  0001 C CNN
 F 1 "GND" H 5700 5250 50  0000 C CNN
 F 2 "" H 5700 5400 50  0001 C CNN
@@
 F 0 "U1" H 5100 5700 60  0000 C CNN
 F 1 "NUP2105LT1G" H 5100 4900 60  0000 C CNN
-F 2 "footprints:SC-59_Handsoldering" H 5100 5300 60  0001 C CNN
+F 2 "footprints:SOT23_NPN" H 5100 5300 60  0001 C CNN
 F 3 "NUP2105L-D-771105.pdf" H 5100 5300 60  0001 C CNN
 F 4 "ON Semiconductor" H 5100 5300 60  0001 C CNN "Manf"
@@
 	5700 5300 5700 5400
 $Comp
-L GND #PWR020
+L GND #PWR019
 U 1 1 594C7F7D
 P 6650 4150
-F 0 "#PWR020" H 6650 3900 50  0001 C CNN
+F 0 "#PWR019" H 6650 3900 50  0001 C CNN
 F 1 "GND" H 6650 4000 50  0000 C CNN
 F 2 "" H 6650 4150 50  0001 C CNN
@@
 $EndComp
 $Comp
-L GND #PWR021
+L GND #PWR020
 U 1 1 594C96DB
 P 8400 6050
-F 0 "#PWR021" H 8400 5800 50  0001 C CNN
+F 0 "#PWR020" H 8400 5800 50  0001 C CNN
 F 1 "GND" H 8400 5900 50  0000 C CNN
 F 2 "" H 8400 6050 50  0001 C CNN
@@
 	9700 6350 3400 6350
 $Comp
-L GNDA #PWR022
+L GNDA #PWR021
 U 1 1 5962D076
 P 4200 2800
-F 0 "#PWR022" H 4200 2550 50  0001 C CNN
+F 0 "#PWR021" H 4200 2550 50  0001 C CNN
 F 1 "GNDA" H 4200 2650 50  0000 C CNN
 F 2 "" H 4200 2800 50  0001 C CNN
@@
 $EndComp
 $Comp
-L +3V3 #PWR023
+L +3V3 #PWR022
 U 1 1 596C91FD
 P 8400 5250
-F 0 "#PWR023" H 8400 5100 50  0001 C CNN
+F 0 "#PWR022" H 8400 5100 50  0001 C CNN
 F 1 "+3V3" H 8400 5390 50  0000 C CNN
 F 2 "" H 8400 5250 50  0001 C CNN
@@
 $EndComp
 $Comp
-L +5V #PWR024
+L +5V #PWR023
 U 1 1 596C9B94
 P 5100 1000
-F 0 "#PWR024" H 5100 850 50  0001 C CNN
+F 0 "#PWR023" H 5100 850 50  0001 C CNN
 F 1 "+5V" H 5100 1140 50  0000 C CNN
 F 2 "" H 5100 1000 50  0001 C CNN
